File: Generation2/TofBreakoutBoardDesign/VL53L8CXBreakoutBoardSchematic.kicad_pcb (KiCad board)
At the start: 2 copper layers, 24 parts, among them J1 JST Connector, U1 VL53L8CX, U2 NXS0108, U3 AP2112K-1.8

Commit message: Reorganize KiCad libraries and update footprint assignments
Parts:
- U1: footprint VL53L8CX:IC17_LGA16_STM -> VL53L8CX:VL53L8CX
- U2: footprint NXS0108:TSSOP20_SOT360-1_NEX -> NXS0108:NXS0108
Changed lines of the file:
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@@
 		)
 	)
-	(footprint "VL53L8CX:IC17_LGA16_STM"
+	(footprint "VL53L8CX:VL53L8CX"
 		(layer "F.Cu")
 		(at 148.5 73.557501)
@@
 		)
 	)
-	(footprint "NXS0108:TSSOP20_SOT360-1_NEX"
+	(footprint "NXS0108:NXS0108"
 		(layer "F.Cu")
 		(at 140.5 89)
