File: Generation2/TofBreakoutBoardDesign/VL53L8CXBreakoutBoardSchematic.kicad_sch (KiCad schematic)
At the start: 24 parts, among them J1 JST Connector, U1 VL53L8CX, U2 NXS0108, U3 AP2112K-1.8

Commit message: Reorganize KiCad libraries and update footprint assignments
Parts:
- U1: footprint VL53L8CX:IC17_LGA16_STM -> VL53L8CX:VL53L8CX
- U2: footprint NXS0108:TSSOP20_SOT360-1_NEX -> NXS0108:NXS0108
Connections:
- net LPnLV: now reaches R5.2, U1.A2 (LPN), U2.5 (A4)
- no-connect marks 0 -> 1
